File: SQRL-Carrier.kicad_pcb (KiCad board)
At the start: 4 copper layers, 100 x 78 mm, 59 parts, among them J1 M.2_M-key, J2 PCIE-164-02-F-D-RA, J3 4-Pin Molex, U1 DSC1104, U2 SI53322, U3 TPS563231, U4 TPS563231, U5 spoolqueue_logo

Commit message: Hardware revision 2
Parts:
- added C9: 1μF, Capacitor_SMD:C_0402_1005Metric, F.Cu at (142.3, 85.7)
- added R23: 475Ω, Resistor_SMD:R_0402_1005Metric, F.Cu at (141.8, 79.3)
- added REF**: alignment_pin, SQRL-Carrier:alignment_pin, F.Cu at (149.0, 123.5)
- added REF**: alignment_pin, SQRL-Carrier:alignment_pin, F.Cu at (71.0, 54.5)
- U2: value SI53322 -> SY75572L; footprint Package_DFN_QFN:VQFN-16-1EP_3x3mm_P0.5mm_EP1.68x1.68mm_ThermalVias -> Package_DFN_QFN:VQFN-16-1EP_3x3mm_P0.5mm_EP1.45x1.45mm
- moved R1 8.49 mm to (136.7, 87.4)
- moved R2 8.49 mm to (136.7, 85.4)
- moved R3 8.49 mm to (138.8, 86.9)
- moved R4 8.49 mm to (138.8, 85.9)
- moved C5 6.96 mm to (139.1, 82.7)
- moved R12 4.83 mm to (137.8, 77.4)
- moved R13 4.83 mm to (139.8, 77.4)
- moved R8 4.83 mm to (138.3, 79.5)
- moved R9 4.83 mm to (139.3, 79.5)
- moved U2 1.00 mm to (142.1, 82.7), turned to 180 degrees
Connections:
- U2 pad 1: GND -> /CLK-
- U2 pad 10: /Q0- -> +3V3_PCIe
- U2 pad 11: /Q1+ -> GND
- U2 pad 12: /Q1- -> /Q1+
- U2 pad 13: Net-(U2-Pad13) -> /Q1-
- U2 pad 15: Net-(U2-Pad15) -> +3V3_PCIe
- U2 pad 16: Net-(U2-Pad16) -> /CLK+
- U2 pad 17: GND -> (no net)
- U2 pad 5: +3V3_PCIe -> Net-(U2-Pad5)
- U2 pad 6: /CLK+ -> GND
- U2 pad 7: /CLK- -> Net-(R23-Pad1)
- U2 pad 8: Net-(U2-Pad8) -> /Q0+
- U2 pad 9: /Q0+ -> /Q0-
Routing:
- net /REFCLK-M.2+: track 82.9 -> 74.0 mm
- net /REFCLK-M.2-: track 82.9 -> 74.0 mm
- net +3V3_PCIe: track 32.0 -> 38.1 mm, vias 10 -> 28
- net GND: track 85.3 -> 90.6 mm, vias 228 -> 99
- net /CLK+: track 4.58 -> 8.56 mm
- net /CLK-: track 4.58 -> 8.37 mm
- net /Q0-: track 1.89 -> 3.59 mm
- net /Q0+: track 1.89 -> 3.40 mm
- net Net-(R23-Pad1): track 0.00 -> 1.50 mm
- net /Q1-: track 3.30 -> 4.26 mm
- net /REFCLK-16-: track 11.6 -> 10.9 mm
- net /REFCLK-16+: track 11.6 -> 11.0 mm
- net +3V3_M.2: vias 18 -> 33
Other:
- board text added: "S/N:"
